Commit message: delete gps color material

File: catkin_ws/src/vmrc/robotx_gazebo/urdf/wamv_gazebo_gps_plugin.xacro (robot description, xacro)
@@ -7,7 +7,4 @@
         <geometry>
           <box size="0.2 1.4 0.2" />
-          <material name="Green">
-          	<color rgba="0 1.0 0.0 1.0"/>
-          </material>
         </geometry>
       </visual>

Commit message: fix coordinate and tf and frame

File: catkin_ws/src/vmrc/robotx_gazebo/urdf/wamv_gazebo_gps_plugin.xacro (robot description, xacro)
@@ -18,5 +18,5 @@
 		<updateRate>5.0</updateRate>
 		<alwaysOn>true</alwaysOn>
-	        <bodyName>${name}</bodyName>
+	        <bodyName>gps</bodyName>
 	        <frameId>gps</frameId>
 		<topicName>gps</topicName>

File: catkin_ws/src/vmrc/wamv_description/urdf/wamv_robotx_nctu.xacro (robot description, xacro)
@@ -25,5 +25,5 @@
       <xacro:include filename="$(find robotx_gazebo)/urdf/wamv_gazebo_lidar_plugin.xacro" />
       <xacro:wamv_HDL32E_lidar parent="base_link" name="velodyne" topic="/velodyne_points" hz="8" samples="1800" min_range="0" max_range="50.0" min_angle="-3.14" max_angle="3.14" noise="0.01">
-        <origin xyz="0.3 0 1.8" rpy="0 0 3.14" />
+        <origin xyz="0.3 0 1.8" rpy="0 0 -1.57" />
       </xacro:wamv_HDL32E_lidar>
   </xacro:if>
@@ -31,5 +31,5 @@
   <xacro:if value="$(arg gps)">
       <xacro:include filename="$(find robotx_gazebo)/urdf/wamv_gazebo_gps_plugin.xacro" />
-      <xacro:wamv_gps name="wamv_gps" latitude="21.30996" longitude="-157.8901" altitude="2.5">
+      <xacro:wamv_gps name="gps" latitude="21.30996" longitude="-157.8901" altitude="2.5">
         <origin xyz="0.2 0.0 2.5" rpy="0 0 0" />
       </xacro:wamv_gps>
@@ -38,5 +38,5 @@
   <xacro:if value="$(arg imu)">
       <xacro:include filename="$(find robotx_gazebo)/urdf/wamv_gazebo_imu_plugin.xacro" />
-      <xacro:wamv_imu name="wamv_imu">
+      <xacro:wamv_imu name="imu">
       </xacro:wamv_imu>
   </xacro:if>
