Commit message: add imu tf

File: catkin_ws/src/vmrc/robotx_gazebo/urdf/wamv_gazebo_imu_plugin.xacro (robot description, xacro)
@@ -1,5 +1,17 @@
 <?xml version="1.0"?>
 <robot xmlns:xacro="http://ros.org/wiki/xacro">
-  <xacro:macro name="wamv_imu" params="name">
+  <xacro:macro name="wamv_imu" params="*origin name">
+    <link name="${name}">
+      <visual>
+        <geometry>
+          <box size="0.1 0.1 0.1" />
+        </geometry>
+      </visual>
+    </link>
+    <joint name="${name}_joint" type="fixed">
+      <xacro:insert_block name="origin"/>
+      <parent link="base_link"/>
+      <child link="${name}"/>
+    </joint>
     <gazebo>
       <!-- Either plugin should work -->

File: catkin_ws/src/vmrc/wamv_description/urdf/wamv_robotx_nctu.xacro (robot description, xacro)
@@ -31,5 +31,5 @@
   <xacro:if value="$(arg gps)">
       <xacro:include filename="$(find robotx_gazebo)/urdf/wamv_gazebo_gps_plugin.xacro" />
-      <xacro:wamv_gps name="gps" latitude="21.30996" longitude="-157.8901" altitude="2.5">
+      <xacro:wamv_gps name="gps" latitude="21.30996" longitude="-157.8901"  altitude="2.5">
         <origin xyz="0.2 0.0 2.5" rpy="0 0 0" />
       </xacro:wamv_gps>
@@ -39,4 +39,5 @@
       <xacro:include filename="$(find robotx_gazebo)/urdf/wamv_gazebo_imu_plugin.xacro" />
       <xacro:wamv_imu name="imu">
+        <origin xyz="0.2 0.0 2.0" rpy="0 0 0" />
       </xacro:wamv_imu>
   </xacro:if>
