Commit message: change the location of cameras

File: catkin_ws/src/vmrc/robotx_gazebo/urdf/wamv_gazebo_front_camera_plugin.xacro (robot description, xacro)
@@ -4,8 +4,8 @@
   <!-- camera position -->
   <xacro:property name="origin_left">
-    <origin xyz="0.65 -0.2 1.45" rpy="0 0 0" />
+    <origin xyz="0.65 -0.3 1.45" rpy="0 0 0" />
   </xacro:property>
   <xacro:property name="origin_right">
-    <origin xyz="0.65 0.2 1.45" rpy="0 0 0" />
+    <origin xyz="0.65 0.3 1.45" rpy="0 0 0" />
   </xacro:property>
   <!-- left camera -->

Commit message: update new camera angle

File: catkin_ws/src/vmrc/robotx_gazebo/urdf/wamv_gazebo_front_camera_plugin.xacro (robot description, xacro)
@@ -4,8 +4,11 @@
   <!-- camera position -->
   <xacro:property name="origin_left">
-    <origin xyz="0.65 -0.3 1.45" rpy="0 0 0" />
+    <origin xyz="0.65 -0.3 1.6" rpy="0 0 -0.785" />
   </xacro:property>
   <xacro:property name="origin_right">
-    <origin xyz="0.65 0.3 1.45" rpy="0 0 0" />
+    <origin xyz="0.65 0.3 1.6" rpy="0 0 0.785" />
+  </xacro:property>
+  <xacro:property name="origin_mid">
+    <origin xyz="0.65 0 1.6" rpy="0 0 0" />
   </xacro:property>
   <!-- left camera -->
@@ -25,5 +28,5 @@
   <gazebo reference="left_front_camera_link">
     <sensor type="camera" name="left_camera">
-      <update_rate>30.0</update_rate>
+      <update_rate>10.0</update_rate>
       <camera name="head">
         <horizontal_fov>1.3962634</horizontal_fov>
@@ -49,8 +52,8 @@
         <alwaysOn>true</alwaysOn>
         <updateRate>0.0</updateRate>
-        <cameraName>camera/left_front</cameraName>
-        <imageTopicName>image_raw</imageTopicName>
+        <cameraName>zed1/rgb</cameraName>
+        <imageTopicName>image_rect</imageTopicName>
         <cameraInfoTopicName>camera_info</cameraInfoTopicName>
-        <frameName>left_front_camera</frameName>
+        <frameName>zed1</frameName>
         <hackBaseline>0.07</hackBaseline>
         <distortionK1>0.0</distortionK1>
@@ -78,5 +81,5 @@
   <gazebo reference="right_front_camera_link">
     <sensor type="camera" name="right_camera">
-      <update_rate>30.0</update_rate>
+      <update_rate>10.0</update_rate>
       <camera name="head">
         <horizontal_fov>1.3962634</horizontal_fov>
@@ -102,8 +105,61 @@
         <alwaysOn>true</alwaysOn>
         <updateRate>0.0</updateRate>
-        <cameraName>camera/right_front</cameraName>
-        <imageTopicName>image_raw</imageTopicName>
+        <cameraName>zed3/rgb</cameraName>
+        <imageTopicName>image_rect</imageTopicName>
         <cameraInfoTopicName>camera_info</cameraInfoTopicName>
-        <frameName>right_front_camera</frameName>
+        <frameName>zed3</frameName>
+        <hackBaseline>0.07</hackBaseline>
+        <distortionK1>0.0</distortionK1>
+        <distortionK2>0.0</distortionK2>
+        <distortionK3>0.0</distortionK3>
+        <distortionT1>0.0</distortionT1>
+        <distortionT2>0.0</distortionT2>
+      </plugin>
+    </sensor>
+  </gazebo>
+  <!-- mid camera -->
+  <link name="mid_front_camera_link">
+    <visual>
+      <origin xyz="-0.01 0 0" rpy="1.57 0 1.57"/>
+      <geometry>
+        <mesh filename="model://zed/zed_model.dae" scale="0.02 0.02 0.02"/>
+      </geometry>
+    </visual>
+  </link>
+  <joint name="mid_front_camera_joint" type="fixed">
+    <xacro:insert_block name="origin_mid" />
+    <parent link="base_link"/>
+    <child link="mid_front_camera_link"/>
+  </joint>
+  <gazebo reference="mid_front_camera_link">
+    <sensor type="camera" name="mid_camera">
+      <update_rate>10.0</update_rate>
+      <camera name="head">
+        <horizontal_fov>1.3962634</horizontal_fov>
+        <image>
+          <width>1280</width>
+          <height>720</height>
+          <format>R8G8B8</format>
+        </image>
+        <clip>
+          <near>0.02</near>
+          <far>300</far>
+        </clip>
+        <noise>
+          <type>gaussian</type>
+          <!-- Noise is sampled independently per pixel on each frame.
+               That pixel's noise value is added to each of its color
+               channels, which at that point lie in the range [0,1]. -->
+          <mean>0.0</mean>
+          <stddev>0.007</stddev>
+        </noise>
+      </camera>
+      <plugin name="camera_controller_front_right_front_camera" filename="libgazebo_ros_camera.so">
+        <alwaysOn>true</alwaysOn>
+        <updateRate>0.0</updateRate>
+        <cameraName>zed2/rgb</cameraName>
+        <imageTopicName>image_rect</imageTopicName>
+        <cameraInfoTopicName>camera_info</cameraInfoTopicName>
+        <frameName>zed2</frameName>
         <hackBaseline>0.07</hackBaseline>
         <distortionK1>0.0</distortionK1>

File: catkin_ws/src/vmrc/wamv_description/urdf/wamv_robotx_nctu.xacro (robot description, xacro)
@@ -24,5 +24,5 @@
   <xacro:if value="$(arg lidar)">
       <xacro:include filename="$(find robotx_gazebo)/urdf/wamv_gazebo_lidar_plugin.xacro" />
-      <xacro:wamv_HDL32E_lidar parent="base_link" name="velodyne" topic="/velodyne_points" hz="7" samples="600" min_range="1" max_range="50.0" min_angle="0" max_angle="3.14" noise="0.01">
+      <xacro:wamv_HDL32E_lidar parent="base_link" name="velodyne" topic="/velodyne_points" hz="7" samples="600" min_range="0" max_range="50.0" min_angle="-3.14" max_angle="3.14" noise="0.01">
         <origin xyz="0.3 0 1.8" rpy="0 0 -1.57" />
       </xacro:wamv_HDL32E_lidar>

Commit message: rename zed and position

File: catkin_ws/src/vmrc/robotx_gazebo/urdf/wamv_gazebo_front_camera_plugin.xacro (robot description, xacro)
@@ -4,11 +4,11 @@
   <!-- camera position -->
   <xacro:property name="origin_left">
+    <origin xyz="0.65 0.3 1.6" rpy="0 0 0.785" />
+  </xacro:property>
+  <xacro:property name="origin_right">
     <origin xyz="0.65 -0.3 1.6" rpy="0 0 -0.785" />
   </xacro:property>
-  <xacro:property name="origin_right">
-    <origin xyz="0.65 0.3 1.6" rpy="0 0 0.785" />
-  </xacro:property>
   <xacro:property name="origin_mid">
-    <origin xyz="0.65 0 1.6" rpy="0 0 0" />
+    <origin xyz="0.65 0 1.6" rpy="-3.14 0 0" />
   </xacro:property>
   <!-- left camera -->
@@ -52,8 +52,8 @@
         <alwaysOn>true</alwaysOn>
         <updateRate>0.0</updateRate>
-        <cameraName>zed1/rgb</cameraName>
+        <cameraName>zed_left/rgb</cameraName>
         <imageTopicName>image_rect_color</imageTopicName>
         <cameraInfoTopicName>camera_info</cameraInfoTopicName>
-        <frameName>zed1</frameName>
+        <frameName>zed_left</frameName>
         <hackBaseline>0.07</hackBaseline>
         <distortionK1>0.0</distortionK1>
@@ -105,8 +105,8 @@
         <alwaysOn>true</alwaysOn>
         <updateRate>0.0</updateRate>
-        <cameraName>zed3/rgb</cameraName>
+        <cameraName>zed_right/rgb</cameraName>
         <imageTopicName>image_rect_color</imageTopicName>
         <cameraInfoTopicName>camera_info</cameraInfoTopicName>
-        <frameName>zed3</frameName>
+        <frameName>zed_right</frameName>
         <hackBaseline>0.07</hackBaseline>
         <distortionK1>0.0</distortionK1>
@@ -158,8 +158,8 @@
         <alwaysOn>true</alwaysOn>
         <updateRate>0.0</updateRate>
-        <cameraName>zed2/rgb</cameraName>
+        <cameraName>zed_mid/rgb</cameraName>
         <imageTopicName>image_rect_color</imageTopicName>
         <cameraInfoTopicName>camera_info</cameraInfoTopicName>
-        <frameName>zed2</frameName>
+        <frameName>zed_mid</frameName>
         <hackBaseline>0.07</hackBaseline>
         <distortionK1>0.0</distortionK1>

Commit message: Invert mid camera

File: catkin_ws/src/vmrc/robotx_gazebo/urdf/wamv_gazebo_front_camera_plugin.xacro (robot description, xacro)
@@ -10,5 +10,5 @@
   </xacro:property>
   <xacro:property name="origin_mid">
-    <origin xyz="0.65 0 1.6" rpy="-3.14 0 0" />
+    <origin xyz="0.65 0 1.6" rpy="0 0 0" />
   </xacro:property>
   <!-- left camera -->

Commit message: add watchtower urdf and revise camera plugin with robot name topic

File: catkin_ws/src/vmrc/robotx_gazebo/urdf/wamv_gazebo_front_camera_plugin.xacro (robot description, xacro)
@@ -1,5 +1,5 @@
 <?xml version="1.0"?>
 <robot xmlns:xacro="http://ros.org/wiki/xacro">
-  <xacro:macro name="wamv_front_camera" params="name">
+  <xacro:macro name="wamv_front_camera" params="name robot_name:=/ ">
   <!-- camera position -->
   <xacro:property name="origin_left">
@@ -52,5 +52,5 @@
         <alwaysOn>true</alwaysOn>
         <updateRate>0.0</updateRate>
-        <cameraName>zed_left/rgb</cameraName>
+        <cameraName>${robot_name}/zed_left/rgb</cameraName>
         <imageTopicName>image_rect_color</imageTopicName>
         <cameraInfoTopicName>camera_info</cameraInfoTopicName>
@@ -105,5 +105,5 @@
         <alwaysOn>true</alwaysOn>
         <updateRate>0.0</updateRate>
-        <cameraName>zed_right/rgb</cameraName>
+        <cameraName>${robot_name}/zed_right/rgb</cameraName>
         <imageTopicName>image_rect_color</imageTopicName>
         <cameraInfoTopicName>camera_info</cameraInfoTopicName>
@@ -158,5 +158,5 @@
         <alwaysOn>true</alwaysOn>
         <updateRate>0.0</updateRate>
-        <cameraName>zed_mid/rgb</cameraName>
+        <cameraName>${robot_name}/zed_mid/rgb</cameraName>
         <imageTopicName>image_rect_color</imageTopicName>
         <cameraInfoTopicName>camera_info</cameraInfoTopicName>
