Commit message: fix apriltag size and remove lidar pulgin of watchtower

File: catkin_ws/src/vmrc/robotx_gazebo/urdf/wamv_gazebo_apriltags_plugin.xacro (robot description, xacro)
@@ -1,7 +1,7 @@
 <?xml version="1.0"?>
 <robot xmlns:xacro="http://ros.org/wiki/xacro">
-  <xacro:macro name="wamv_apriltags" params="*origin name longitude:=-157.8901 latitude:=21.30996 altitude:=1.5">
-  <xacro:arg name="tag_id" default="0"/>
-  <xacro:arg name="tag_size" default="0.54"/>
+  <xacro:macro name="wamv_apriltags" params="*origin name longitude:=-157.8901 latitude:=21.30996 altitude:=1.5 tag_id:=0 tag_size:=0.54">
+  <!--xacro:arg name="tag_id" default="0"/-->
+  <xacro:property name="size" value="${tag_size}"/>
     <link name="${name}">
         <gravity>0</gravity>
@@ -25,5 +25,5 @@
                 rpy="0 0 0" />
             <geometry>
-                <box size="0.01 $(arg tag_size) $(arg tag_size)"/>
+                <box size="0.01 ${size} ${size}"/>
             </geometry>
             <!--<material name="Hope"/>-->
@@ -34,5 +34,6 @@
                 rpy="0 0 0" />
             <geometry>
-                <box size="0.01 $(arg tag_size) $(arg tag_size)"/>
+                <box size="0.01 ${size} ${size}"/>
+                <!--box size="0.01 $(arg tag_size) $(arg tag_size)"/-->
             </geometry>
         </collision>
@@ -45,5 +46,5 @@
     <gazebo reference="${name}">
         <turnGravityOff>true</turnGravityOff>
-        <material>a_$(arg tag_id)/Image</material>
+        <material>a_${tag_id}/Image</material>
     </gazebo>
   </xacro:macro>

File: catkin_ws/src/vmrc/wamv_description/urdf/wamv_robotx_nctu.xacro (robot description, xacro)
@@ -51,6 +51,14 @@
   <xacro:if value="$(arg apriltags)">
       <xacro:include filename="$(find robotx_gazebo)/urdf/wamv_gazebo_apriltags_plugin.xacro" />
-      <xacro:wamv_apriltags name="wamv_apriltags">
-        <origin xyz="-0.95 0.0 1.0" rpy="0 0 0" />
+      <xacro:wamv_apriltags name="wamv_right_apriltag" tag_id="2" tag_size="0.80">
+        <origin xyz="-0.45 -0.5 1.5" rpy="0 0 -1.57079"/>
+      </xacro:wamv_apriltags>
+      <xacro:include filename="$(find robotx_gazebo)/urdf/wamv_gazebo_apriltags_plugin.xacro" />
+      <xacro:wamv_apriltags name="wamv_back_apriltag" tag_id="1" tag_size="0.80">
+        <origin xyz="-0.95 0.0 1.5" rpy="0 0 0"/>
+      </xacro:wamv_apriltags>
+      <xacro:include filename="$(find robotx_gazebo)/urdf/wamv_gazebo_apriltags_plugin.xacro" />
+      <xacro:wamv_apriltags name="wamv_left_apriltag" tag_id="0" tag_size="0.80">
+        <origin xyz="-0.45 0.5 1.5" rpy="0 0 1.57079"/>
       </xacro:wamv_apriltags>
   </xacro:if>
