Commit message: add two different id tag to apriltag_float

File: catkin_ws/src/vmrc/robotx_gazebo/urdf/watchtower_gazebo_camera_plugin.xacro (robot description, xacro)
@@ -24,5 +24,6 @@
       <update_rate>10.0</update_rate>
       <camera name="head">
-        <horizontal_fov>1.3962634</horizontal_fov>
+        <!--<horizontal_fov>1.3962634</horizontal_fov>-->
+        <horizontal_fov>1.57</horizontal_fov>
         <image>
           <width>1280</width>

File: catkin_ws/src/vmrc/wamv_description/urdf/apriltag.xacro (robot description, xacro)
@@ -4,5 +4,5 @@
   <!-- Defines the base vehicle -->
   <xacro:include filename="$(find wamv_description)/urdf/apriltag_base.xacro" />
-  <xacro:apriltag_base name="$(arg robot_name)_apriltag_base_plugin" tag_id="$(arg tag_id)" tag_size="$(arg tag_size)"/>
+  <xacro:apriltag_base name="$(arg robot_name)_apriltag_base_plugin" tag_id="$(arg tag_id)" tag_id2="$(arg tag_id2)" tag_size="$(arg tag_size)"/>
   <!-- Attach hydrodynamics plugin -->
   <xacro:include filename="$(find robotx_gazebo)/urdf/wamv_gazebo_dynamics_plugin.xacro" />

File: catkin_ws/src/vmrc/wamv_description/urdf/apriltag_base.xacro (robot description, xacro)
@@ -1,5 +1,5 @@
 <?xml version="1.0"?>
 <robot xmlns:xacro="http://ros.org/wiki/xacro">
-  <xacro:macro name="apriltag_base" params=" name tag_id:=0 tag_size:=0.8">
+  <xacro:macro name="apriltag_base" params=" name tag_id:=0 tag_id2:=0 tag_size:=0.8">
   <xacro:property name="size" value="${tag_size}"/>
 <!--
@@ -94,5 +94,5 @@
   <gazebo reference="apriltag_1">
     <turnGravityOff>false</turnGravityOff>
-    <material>a_${tag_id}/Image</material>
+    <material>a_${tag_id2}/Image</material>
   </gazebo>
   <gazebo reference="apriltag_2">

File: catkin_ws/src/vmrc/wamv_description/urdf/wamv_robotx_nctu.xacro (robot description, xacro)
@@ -51,13 +51,14 @@
   <xacro:if value="$(arg apriltags)">
       <xacro:include filename="$(find robotx_gazebo)/urdf/wamv_gazebo_apriltags_plugin.xacro" />
-      <xacro:wamv_apriltags name="wamv_right_apriltag" tag_id="2" tag_size="0.80">
+      <xacro:wamv_apriltags name="wamv_right_apriltag" tag_id="503" tag_size="1.00">
         <origin xyz="-0.45 -0.5 1.5" rpy="0 0 -1.57079"/>
       </xacro:wamv_apriltags>
+502
       <xacro:include filename="$(find robotx_gazebo)/urdf/wamv_gazebo_apriltags_plugin.xacro" />
-      <xacro:wamv_apriltags name="wamv_back_apriltag" tag_id="1" tag_size="0.80">
+      <xacro:wamv_apriltags name="wamv_back_apriltag" tag_id="502" tag_size="1.00">
         <origin xyz="-0.95 0.0 1.5" rpy="0 0 0"/>
       </xacro:wamv_apriltags>
       <xacro:include filename="$(find robotx_gazebo)/urdf/wamv_gazebo_apriltags_plugin.xacro" />
-      <xacro:wamv_apriltags name="wamv_left_apriltag" tag_id="0" tag_size="0.80">
+      <xacro:wamv_apriltags name="wamv_left_apriltag" tag_id="501" tag_size="1.00">
         <origin xyz="-0.45 0.5 1.5" rpy="0 0 1.57079"/>
       </xacro:wamv_apriltags>
