Commit message: revise apriltag base plugin

File: catkin_ws/src/vmrc/wamv_description/urdf/apriltag.xacro (robot description, xacro)
@@ -1,7 +1,8 @@
 <?xml version="1.0"?>
 <robot xmlns:xacro="http://ros.org/wiki/xacro"
-       name="apriltage">
+       name="apriltag">
   <!-- Defines the base vehicle -->
   <xacro:include filename="$(find wamv_description)/urdf/apriltag_base.xacro" />
+  <xacro:apriltag_base name="$(arg robot_name)_apriltag_base_plugin" tag_id="$(arg tag_id)" tag_size="$(arg tag_size)"/>
   <!-- Attach hydrodynamics plugin -->
   <xacro:include filename="$(find robotx_gazebo)/urdf/wamv_gazebo_dynamics_plugin.xacro" />

File: catkin_ws/src/vmrc/wamv_description/urdf/apriltag_base.xacro (robot description, xacro)
@@ -1,9 +1,6 @@
 <?xml version="1.0"?>
-<robot name="apriltag"
-       xmlns:xacro="http://ros.org/wiki/xacro">
-<!--
-  <xacro:macro name="apriltag" params="tag_id:=0 tag_size:=0.8">
-  <xacro:property name="tag_size" value="${tag_size}"/>
--->
+<robot xmlns:xacro="http://ros.org/wiki/xacro">
+  <xacro:macro name="apriltag_base" params=" name tag_id:=0 tag_size:=0.8">
+  <xacro:property name="size" value="${tag_size}"/>
 <!--
   <xacro:property name="tag_size" value="0.7" />
@@ -14,5 +11,5 @@
   <link name="base_link">
     <inertial>
-      <origin xyz="0 0 1" rpy="0 0 0"/>
+      <origin xyz="0 0 0.25" rpy="0 0 0"/>
       <mass value="1"/>
       <inertia
@@ -23,5 +20,5 @@
     <visual>
       <origin
-        xyz="0 0 1"
+        xyz="0 0 0.25"
         rpy="0 0 0" />
       <geometry>
@@ -31,5 +28,5 @@
     <collision>
       <origin
-        xyz="0 0 1"
+        xyz="0 0 0.25"
         rpy="0 0 0" />
       <geometry>
@@ -41,17 +38,17 @@
   <link name="apriltag_1">
     <collision>
-      <origin xyz="0 0 1" rpy="0 0 0"/>
+      <origin xyz="-0.25 -0.25 0.75" rpy="0 0 0"/>
       <geometry>
-        <box size="0.01 0.7 0.7"/>
+        <box size="0.01 ${size} ${size}"/>
       </geometry>
     </collision>
     <visual>
-      <origin xyz="0 0 1" rpy="0 0 0"/>
+      <origin xyz="-0.25 -0.25 0.75" rpy="0 0 0"/>
       <geometry>
-        <box size="0.01 0.7 0.7"/>
+        <box size="0.01 ${size} ${size}"/>
       </geometry>
     </visual>
     <inertial>
-      <origin xyz="0 0 1" rpy="0 0 0"/>
+      <origin xyz="-0.25 -0.25 0.75" rpy="0 0 0"/>
       <mass value="1"/>
       <inertia
@@ -64,18 +61,18 @@
   <link name="apriltag_2">
     <collision>
-      <origin xyz="0 0 1" rpy="0 0 3.14/2"/>
+      <origin xyz="0.25 0.25  0.75" rpy="0 0 1.57"/>
       <geometry>
-        <box size="0.01 0.54 0.54"/>
+        <box size="0.01 ${size} ${size}"/>
       </geometry>
     </collision>
     <visual>
-      <origin xyz="0 0 1" rpy="0 0 3.14/2"/>
+      <origin xyz="0.25 0.25  0.75" rpy="0 0 1.57"/>
       <geometry>
-        <box size="0.01 0.54 0.54"/>
+        <box size="0.01 ${size} ${size}"/>
       </geometry>
       <material name="orange"/>
     </visual>
     <inertial>
-      <origin xyz="0 0 1" rpy="0 0 3.14/2"/>
+      <origin xyz="0.25 0.25  0.75" rpy="0 0 1.57"/>
       <mass value="1"/>
       <inertia
@@ -97,10 +94,10 @@
   <gazebo reference="apriltag_1">
     <turnGravityOff>false</turnGravityOff>
-    <material>a_0/Image</material>
+    <material>a_${tag_id}/Image</material>
   </gazebo>
   <gazebo reference="apriltag_2">
     <turnGravityOff>false</turnGravityOff>
-    <material>a_1/Image</material>
+    <material>a_${tag_id}/Image</material>
   </gazebo>
-  <!--</xacro:macro> -->
+  </xacro:macro>
 </robot>
