Commit message: update duckieboat setting in gazebo

File: catkin_ws/src/vmrc/wamv_description/urdf/duckieboat.xacro (robot description, xacro)
@@ -1,19 +1,22 @@
 <?xml version="1.0"?>
 <robot xmlns:xacro="http://ros.org/wiki/xacro"
-       name="watchtower">
+       name="duckieboat">
   <!-- Defines the base vehicle -->
   <xacro:include filename="$(find wamv_description)/urdf/duckieboat_base.xacro" />
   <!-- Attach hydrodynamics plugin -->
   <xacro:include filename="$(find robotx_gazebo)/urdf/wamv_gazebo_dynamics_plugin.xacro" />
-  <xacro:usv_dynamics_gazebo name="$(arg robot_name)_dynamics_plugin"/>
+  <xacro:usv_dynamics_gazebo name="duckieboat_dynamics_plugin"/>
   <!-- Attach wind plugin -->
   <xacro:if value="$(arg wind)">
       <xacro:include filename="$(find robotx_gazebo)/urdf/wamv_gazebo_wind_plugin.xacro" />
-      <xacro:usv_wind_gazebo name="$(arg robot_name)_wind_plugin"/>
+      <xacro:usv_wind_gazebo name="duckieboat_wind_plugin"/>
   </xacro:if>
+  <!-- Attach thrust plugin -->
+  <xacro:include filename="$(find robotx_gazebo)/urdf/wamv_gazebo_thrust_plugin.xacro" />
+  <xacro:usv_thrust_gazebo name="duckieboat_thrust_plugin"/>
   <!-- Attach front camera plugin -->
-  <xacro:include filename="$(find robotx_gazebo)/urdf/watchtower_gazebo_camera_plugin.xacro" />
-      <xacro:watchtower_camera name="$(arg robot_name)_front_camera" robot_name="$(arg robot_name)">
-  </xacro:watchtower_camera>
+  <xacro:include filename="$(find robotx_gazebo)/urdf/duckieboat_gazebo_camera_plugin.xacro" />
+      <xacro:duckieboat_camera name="$(arg robot_name)_front_camera" robot_name="$(arg robot_name)">
+  </xacro:duckieboat_camera>
   <!-- Attach p3d odometry plugin -->
   <xacro:if value="$(arg p3d)">

File: catkin_ws/src/vmrc/wamv_description/urdf/duckieboat_base.xacro (robot description, xacro)
@@ -1,5 +1,5 @@
 <?xml version="1.0"?>
-<robot xmlns:xacro="http://ros.org/wiki/xacro" name="watchtower">
-  <!--<xacro:include filename="properties_watchtower.urdf.xacro"/>-->
+<robot xmlns:xacro="http://ros.org/wiki/xacro" name="duckieboat">
+  <xacro:include filename="propeties_duckieboat.urdf.xacro"/>
   <gazebo reference="base_link">
     <material>Gazebo/Orange</material>
@@ -9,5 +9,5 @@
     <inertial>
       <origin
-        xyz="-0 0 0.5"
+        xyz="0 -0.48 0.5"
         rpy="0 0 0" />
       <mass
@@ -23,5 +23,5 @@
     <visual>
       <origin
-        xyz="0 0 0"
+        xyz="0 -0.48 0"
         rpy="0 0 0" />
       <geometry>
@@ -32,5 +32,5 @@
     <collision>
       <origin
-        xyz="0 0 0"
+        xyz="0 -0.48 0"
         rpy="0 0 0" />
       <geometry>
@@ -40,9 +40,75 @@
     </collision>
   </link>
+  <!-- right motor -->
+  <link name="right_motor">
+    <visual>
+     <geometry>
+       <mesh filename="package://wamv_description/mesh/PROPELLER.dae"/>
+     </geometry>
+    </visual>
+    <collision name="right_motor_collision">
+      <geometry>
+        <mesh filename="package://wamv_description/mesh/PROPELLER.dae"/>
+      </geometry>
+    </collision>
+    <inertial>
+      <mass value="0.01"/>
+      <inertia ixx="0.00086" ixy="0.00" ixz="0.00" iyy="0.00086" iyz="0.00" izz="0.0017"/>
+    </inertial>
+  </link>
+  <joint name="right_motor_joint" type="continuous">
+    <origin xyz="${motor_position_x} -${motor_position_y} ${motor_position_z}"/>
+    <parent link="base_link"/>
+    <child link="right_motor"/>
+    <limit effort="0.5293" velocity="100${pi}" />
+  </joint>
+  <transmission name="right_motor_trans">
+    <type>transmission_interface/SimpleTransmission</type>
+    <joint name="right_motor_joint">
+      <hardwareInterface>VelocityJointInterface</hardwareInterface>
+    </joint>
+    <actuator name="right_motor_actuator">
+      <hardwareInterface>VelocityJointInterface</hardwareInterface>
+      <mechanicalReduction>30</mechanicalReduction>
+    </actuator>
+  </transmission>
+  <!-- left motor -->
+  <link name="left_motor">
+    <visual>
+     <geometry>
+       <mesh filename="package://wamv_description/mesh/PROPELLER.dae"/>
+     </geometry>
+    </visual>
+    <collision name="left_motor_collision">
+      <geometry>
+        <mesh filename="package://wamv_description/mesh/PROPELLER.dae"/>
+      </geometry>
+    </collision>
+    <inertial>
+      <mass value="0.01"/>
+      <inertia ixx="0.00086" ixy="0.00" ixz="0.00" iyy="0.00086" iyz="0.00" izz="0.0017"/>
+    </inertial>
+  </link>
+  <joint name="left_motor_joint" type="continuous">
+    <origin xyz="${motor_position_x} ${motor_position_y} ${motor_position_z}"/>
+    <parent link="base_link"/>
+    <child link="left_motor"/>
+    <limit effort="0.5293" velocity="100${pi}" />
+  </joint>
+  <transmission name="left_motor_trans">
+    <type>transmission_interface/SimpleTransmission</type>
+    <joint name="left_motor_joint">
+      <hardwareInterface>VelocityJointInterface</hardwareInterface>
+    </joint>
+    <actuator name="left_motor_actuator">
+      <hardwareInterface>VelocityJointInterface</hardwareInterface>
+      <mechanicalReduction>30</mechanicalReduction>
+    </actuator>
+  </transmission>
   <joint name="base_link_joint" type="fixed">
     <origin xyz="0 0 0"/>
-    <parent link="base_footprint2"/>
+    <parent link="base_footprint"/>
     <child link="base_link"/>
   </joint>
-  <link name="base_footprint2"/>
+  <link name="base_footprint"/>
 </robot>
