Commit message: add gps xacro on robot

File: catkin_ws/src/vmrc/wamv_description/urdf/wamv_robotx_nctu.xacro (robot description, xacro)
@@ -3,5 +3,5 @@
        name="WAM-V">
   <!-- Defines the base vehicle -->
-  <xacro:include filename="$(find wamv_description)/urdf/wamv_base.xacro" />
+  <xacro:include filename="$(find wamv_description)/urdf/wamv_base_nctu.xacro" />
   <!-- Attach hydrodynamics plugin -->
   <xacro:include filename="$(find robotx_gazebo)/urdf/wamv_gazebo_dynamics_plugin.xacro" />
@@ -23,8 +23,14 @@
   <xacro:if value="$(arg lidar)">
       <xacro:include filename="$(find robotx_gazebo)/urdf/wamv_gazebo_lidar_plugin.xacro" />
-      <xacro:wamv_HDL32E_lidar parent="base_link" name="velodyne" topic="/velodyne_points" hz="10" samples="150" min_range="5" max_range="50.0" min_angle="-1.57" max_angle="1.57" noise="0.1" >
+      <xacro:wamv_HDL32E_lidar parent="base_link" name="velodyne" topic="/velodyne_points" hz="10" samples="220" min_range="5" max_range="50.0" min_angle="-1.57" max_angle="1.57" noise="0.1" >
         <origin xyz="0.5 0 1.3" rpy="0 0 0" />
       </xacro:wamv_HDL32E_lidar>
   </xacro:if>
   <!-- Attach GPS and imu plugin -->
+  <xacro:if value="$(arg gps)">
+      <xacro:include filename="$(find robotx_gazebo)/urdf/wamv_gazebo_gps_plugin.xacro" />
+      <xacro:wamv_gps name="wamv_gps" latitude="21.30996" longitude="-157.8901" altitude="2.5">
+        <origin xyz="0.2 0.0 2.5" rpy="0 0 0" />
+      </xacro:wamv_gps>
+  </xacro:if>
 </robot>

Commit message: fix the lidar problem, remove the sandisland map

File: catkin_ws/src/vmrc/wamv_description/urdf/wamv_robotx_nctu.xacro (robot description, xacro)
@@ -23,12 +23,8 @@
   <!-- Attach LiDAR plugin -->
   <xacro:if value="$(arg lidar)">
-      <!--xacro:include filename="$(find robotx_gazebo)/urdf/wamv_gazebo_lidar_plugin.xacro" />
-      <xacro:wamv_HDL32E_lidar parent="base_link" name="velodyne" topic="/velodyne_points" hz="10" samples="220" min_range="5" max_range="50.0" min_angle="-1.57" max_angle="1.57" noise="0.1">
-        <origin xyz="0.5 0 1.3" rpy="0 0 0" />
-      </xacro:wamv_HDL32E_lidar-->
-      <xacro:include filename="$(find velodyne_description)/urdf/VLP-16.urdf.xacro"/>
-      <VLP-16 parent="base_link" name="velodyne" topic="/velodyne_points">
-        <origin xyz="0.6 0 1.3" rpy="0 0 0" />
-      </VLP-16>
+      <xacro:include filename="$(find robotx_gazebo)/urdf/wamv_gazebo_lidar_plugin.xacro" />
+      <xacro:wamv_HDL32E_lidar parent="base_link" name="velodyne" topic="/velodyne_points" hz="5" samples="500" min_range="5" max_range="50.0" min_angle="-1.57" max_angle="1.57" noise="0.1">
+        <origin xyz="0.3 0 1.8" rpy="0 0 0" />
+      </xacro:wamv_HDL32E_lidar>
   </xacro:if>
   <!-- Attach GPS plugin -->

Commit message: lidar frame equal to real in gazebo

File: catkin_ws/src/vmrc/wamv_description/urdf/wamv_robotx_nctu.xacro (robot description, xacro)
@@ -24,6 +24,6 @@
   <xacro:if value="$(arg lidar)">
       <xacro:include filename="$(find robotx_gazebo)/urdf/wamv_gazebo_lidar_plugin.xacro" />
-      <xacro:wamv_HDL32E_lidar parent="base_link" name="velodyne" topic="/velodyne_points" hz="7" samples="600" min_range="1" max_range="50.0" min_angle="-1.57" max_angle="1.57" noise="0.01">
-        <origin xyz="0.3 0 1.8" rpy="0 0 0" />
+      <xacro:wamv_HDL32E_lidar parent="base_link" name="velodyne" topic="/velodyne_points" hz="7" samples="600" min_range="1" max_range="50.0" min_angle="0" max_angle="3.14" noise="0.01">
+        <origin xyz="0.3 0 1.8" rpy="0 0 -1.57" />
       </xacro:wamv_HDL32E_lidar>
   </xacro:if>

Commit message: fix coordinate and PID

File: catkin_ws/src/vmrc/wamv_description/urdf/wamv_robotx_nctu.xacro (robot description, xacro)
@@ -25,5 +25,5 @@
       <xacro:include filename="$(find robotx_gazebo)/urdf/wamv_gazebo_lidar_plugin.xacro" />
       <xacro:wamv_HDL32E_lidar parent="base_link" name="velodyne" topic="/velodyne_points" hz="8" samples="1800" min_range="0" max_range="50.0" min_angle="-3.14" max_angle="3.14" noise="0.01">
-        <origin xyz="0.3 0 1.8" rpy="0 0 -1.57" />
+        <origin xyz="0.3 0 1.8" rpy="0 0 3.14" />
       </xacro:wamv_HDL32E_lidar>
   </xacro:if>

Commit message: add apriltags on WAM-V

File: catkin_ws/src/vmrc/wamv_description/urdf/wamv_robotx_nctu.xacro (robot description, xacro)
@@ -48,3 +48,10 @@
       </xacro:wamv_p3d>
   </xacro:if>
+  <!-- Attach apriltags -->
+  <xacro:if value="$(arg apriltags)">
+      <xacro:include filename="$(find robotx_gazebo)/urdf/wamv_gazebo_apriltags_plugin.xacro" />
+      <xacro:wamv_apriltags name="wamv_apriltags">
+        <origin xyz="-0.95 0.0 1.0" rpy="0 0 0" />
+      </xacro:wamv_apriltags>
+  </xacro:if>
 </robot>

Commit message: fix wamv apriltag location z+. use gazebo paused=true

File: catkin_ws/src/vmrc/wamv_description/urdf/wamv_robotx_nctu.xacro (robot description, xacro)
@@ -52,14 +52,14 @@
       <xacro:include filename="$(find robotx_gazebo)/urdf/wamv_gazebo_apriltags_plugin.xacro" />
       <xacro:wamv_apriltags name="wamv_right_apriltag" tag_id="503" tag_size="1.00">
-        <origin xyz="-0.45 -0.5 1.5" rpy="0 0 -1.57079"/>
+        <origin xyz="-0.45 -0.5 1.7" rpy="0 0 -1.57079"/>
       </xacro:wamv_apriltags>
 502
       <xacro:include filename="$(find robotx_gazebo)/urdf/wamv_gazebo_apriltags_plugin.xacro" />
       <xacro:wamv_apriltags name="wamv_back_apriltag" tag_id="502" tag_size="1.00">
-        <origin xyz="-0.95 0.0 1.5" rpy="0 0 0"/>
+        <origin xyz="-0.95 0.0 1.7" rpy="0 0 0"/>
       </xacro:wamv_apriltags>
       <xacro:include filename="$(find robotx_gazebo)/urdf/wamv_gazebo_apriltags_plugin.xacro" />
       <xacro:wamv_apriltags name="wamv_left_apriltag" tag_id="501" tag_size="1.00">
-        <origin xyz="-0.45 0.5 1.5" rpy="0 0 1.57079"/>
+        <origin xyz="-0.45 0.5 1.7" rpy="0 0 1.57079"/>
       </xacro:wamv_apriltags>
   </xacro:if>

Commit message: add front apriltag on wamv

File: catkin_ws/src/vmrc/wamv_description/urdf/wamv_robotx_nctu.xacro (robot description, xacro)
@@ -51,4 +51,8 @@
   <xacro:if value="$(arg apriltags)">
       <xacro:include filename="$(find robotx_gazebo)/urdf/wamv_gazebo_apriltags_plugin.xacro" />
+      <xacro:wamv_apriltags name="wamv_front_apriltag" tag_id="512" tag_size="1.00">
+        <origin xyz="1.1 0.0 0.9" rpy="0 0 0"/>
+      </xacro:wamv_apriltags>
+      <xacro:include filename="$(find robotx_gazebo)/urdf/wamv_gazebo_apriltags_plugin.xacro" />
       <xacro:wamv_apriltags name="wamv_right_apriltag" tag_id="503" tag_size="1.00">
         <origin xyz="-0.45 -0.5 1.7" rpy="0 0 -1.57079"/>

Commit message: move side tag to center

File: catkin_ws/src/vmrc/wamv_description/urdf/wamv_robotx_nctu.xacro (robot description, xacro)
@@ -56,5 +56,6 @@
       <xacro:include filename="$(find robotx_gazebo)/urdf/wamv_gazebo_apriltags_plugin.xacro" />
       <xacro:wamv_apriltags name="wamv_right_apriltag" tag_id="503" tag_size="1.00">
-        <origin xyz="-0.45 -0.5 1.7" rpy="0 0 -1.57079"/>
+        <!--origin xyz="-0.45 -0.5 1.7" rpy="0 0 -1.57079"/-->
+        <origin xyz="0 -0.5 1.7" rpy="0 0 -1.57079"/>
       </xacro:wamv_apriltags>
       <xacro:include filename="$(find robotx_gazebo)/urdf/wamv_gazebo_apriltags_plugin.xacro" />
@@ -64,5 +65,6 @@
       <xacro:include filename="$(find robotx_gazebo)/urdf/wamv_gazebo_apriltags_plugin.xacro" />
       <xacro:wamv_apriltags name="wamv_left_apriltag" tag_id="501" tag_size="1.00">
-        <origin xyz="-0.45 0.5 1.7" rpy="0 0 1.57079"/>
+        <!--origin xyz="-0.45 0.5 1.7" rpy="0 0 1.57079"/-->
+        <origin xyz="0 0.5 1.7" rpy="0 0 1.57079"/>
       </xacro:wamv_apriltags>
   </xacro:if>
