Commit message: add apriltag model back color white

File: catkin_ws/src/vmrc/robotx_gazebo/models/apriltag/apriltag.xacro (robot description, xacro)
@@ -41,5 +41,4 @@
   <!-- apriltag_1 -->
   <link name="apriltag_1">
-    <gravity>0</gravity>
     <collision>
       <origin xyz="0 0 0" rpy="0 0 0"/>
@@ -65,5 +64,4 @@
   <!-- apriltag_2 -->
   <link name="apriltag_2">
-    <gravity>0</gravity>
     <collision>
       <origin xyz="0 0 0" rpy="0 0 0"/>
@@ -88,4 +86,22 @@
     </inertial>
   </link>
+  <!-- apriltag_1_back -->
+  <link name="apriltag_1_back">
+    <visual>
+      <origin xyz="-0.24 -0.25 0.75" rpy="0 0 0"/>
+      <geometry>
+        <box size="0.01 ${size} ${size}"/>
+      </geometry>
+    </visual>
+  </link>
+  <!-- apriltag_2_back -->
+  <link name="apriltag_2_back">
+    <visual>
+      <origin xyz="0.25 0.24  0.75" rpy="0 0 1.57"/>
+      <geometry>
+        <box size="0.01 ${size} ${size}"/>
+      </geometry>
+    </visual>
+  </link>
   <!-- joint -->
   <joint name="totem_to_apriltag_1" type="fixed">
@@ -96,4 +112,12 @@
     <parent link="base_link"/>
     <child link="apriltag_2"/>
+  </joint>
+  <joint name="totem_to_apriltag_1_back" type="fixed">
+    <parent link="base_link"/>
+    <child link="apriltag_1_back"/>
+  </joint>
+  <joint name="totem_to_apriltag_2_back" type="fixed">
+    <parent link="base_link"/>
+    <child link="apriltag_2_back"/>
   </joint>
   <!-- apriltage id -->

File: catkin_ws/src/vmrc/robotx_gazebo/urdf/wamv_gazebo_apriltags_plugin.xacro (robot description, xacro)
@@ -5,5 +5,4 @@
   <xacro:property name="size" value="${tag_size}"/>
     <link name="${name}">
-        <gravity>0</gravity>
         <inertial>
             <origin
@@ -39,8 +38,24 @@
         </collision>
     </link>
+    <link name="${name}_back">
+        <visual>
+            <origin
+                xyz="-0.01 0 0"
+                rpy="0 0 0" />
+            <geometry>
+                <box size="0.01 ${size} ${size}"/>
+            </geometry>
+            <!--<material name="Hope"/>-->
+        </visual>
+    </link>
     <joint name="${name}_joint" type="fixed">
       <xacro:insert_block name="origin"/>
       <parent link="base_link"/>
       <child link="${name}"/>
+    </joint>
+    <joint name="${name}_back_joint" type="fixed">
+      <xacro:insert_block name="origin"/>
+      <parent link="base_link"/>
+      <child link="${name}_back"/>
     </joint>
     <gazebo reference="${name}">

File: catkin_ws/src/vmrc/wamv_description/urdf/apriltag_base.xacro (robot description, xacro)
@@ -58,4 +58,13 @@
     </inertial>
   </link>
+  <!-- apriltag_1_back -->
+  <link name="apriltag_1_back">
+    <visual>
+      <origin xyz="-0.24 -0.25 0.75" rpy="0 0 0"/>
+      <geometry>
+        <box size="0.01 ${size} ${size}"/>
+      </geometry>
+    </visual>
+  </link>
   <!-- apriltag_2 -->
   <link name="apriltag_2">
@@ -71,5 +80,4 @@
         <box size="0.01 ${size} ${size}"/>
       </geometry>
-      <material name="orange"/>
     </visual>
     <inertial>
@@ -82,4 +90,13 @@
     </inertial>
   </link>
+  <!-- apriltag_2_back -->
+  <link name="apriltag_2_back">
+    <visual>
+      <origin xyz="0.25 0.24  0.75" rpy="0 0 1.57"/>
+      <geometry>
+        <box size="0.01 ${size} ${size}"/>
+      </geometry>
+    </visual>
+  </link>
   <!-- joint -->
   <joint name="totem_to_apriltag_1" type="fixed">
@@ -87,7 +104,15 @@
     <child link="apriltag_1"/>
   </joint>
+  <joint name="totem_to_apriltag_1_back" type="fixed">
+    <parent link="base_link"/>
+    <child link="apriltag_1_back"/>
+  </joint>
   <joint name="totem_to_apriltag_2" type="fixed">
     <parent link="base_link"/>
     <child link="apriltag_2"/>
+  </joint>
+  <joint name="totem_to_apriltag_2_back" type="fixed">
+    <parent link="base_link"/>
+    <child link="apriltag_2_back"/>
   </joint>
   <!-- apriltage id -->

File: catkin_ws/src/vmrc/wamv_description/urdf/wamv_robotx_nctu.xacro (robot description, xacro)
@@ -54,8 +54,7 @@
         <origin xyz="-0.45 -0.5 1.7" rpy="0 0 -1.57079"/>
       </xacro:wamv_apriltags>
-502
       <xacro:include filename="$(find robotx_gazebo)/urdf/wamv_gazebo_apriltags_plugin.xacro" />
       <xacro:wamv_apriltags name="wamv_back_apriltag" tag_id="502" tag_size="1.00">
-        <origin xyz="-0.95 0.0 1.7" rpy="0 0 0"/>
+        <origin xyz="-0.95 0.0 1.7" rpy="0 0 3.14159"/>
       </xacro:wamv_apriltags>
       <xacro:include filename="$(find robotx_gazebo)/urdf/wamv_gazebo_apriltags_plugin.xacro" />
